File: m_pcb.kicad_pcb (KiCad board)
At the start: 4 copper layers, 142.2 x 134.6 mm, 70 parts, among them J1 tang nano 20k left pins, J10 AudioJack3_Ground, J11 AudioJack3_Ground, J12 Barrel_Jack_MountingPin, J2 tang nano 20k right pins, J3 esp32-p4-pico left pins, J4 esp32-p4-pico right pins, J7 Conn_01x04_Pin, U1 SGTL5000XNLA3, U2 TL072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

Commit message: Update board, readme, image
Parts:
- moved C7 1.11 mm to (128.3, 94.3), turned to 90 degrees
- moved C12 0.76 mm to (113.4, 80.8)
- moved D3 0.55 mm to (171.3, 29.0)
- moved R10 0.54 mm to (132.0, 96.6)
- moved R11 0.54 mm to (129.0, 96.6)
- moved C21 0.30 mm to (168.9, 29.7)
- moved C17 0.12 mm to (132.1, 109.6)
Routing:
- net +9V: track 56.4 -> 45.0 mm
- net Net-(C7-Pad1): track 3.23 -> 1.52 mm
- net I2S_DOUT: track 22.6 -> 21.0 mm
- net Net-(C8-Pad1): track 5.44 -> 6.33 mm
- net Net-(U3A--): track 3.92 -> 4.70 mm
- net Net-(D3-K): track 6.43 -> 5.89 mm
- net GND: vias 76 -> 90
