File: rev-b/electrical/kestrel-revb-mcu.kicad_sch (KiCad schematic)
At the start: 53 parts, among them J701 UART / POWERED TARGET ONLY, SW701 RESET / SMD button MPN pending, SW702 BOOT / SMD button MPN pending, U701 ESP32-P4NRW16X, U702 GD25Q32ESIGR, Y701 40MHz / +/-10ppm / MPN and CL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

Commit message: Route all sixteen RGB source signals with guarded via-in-pad
Connections:
- net MCU_LCD_G6: now also U701.63 (GPIO32); no longer U701.90 (GPIO48)
- net MCU_LCD_R3: now also U701.55 (GPIO26); no longer U701.93 (GPIO50)
- net MCU_LCD_R5: now also U701.57 (GPIO28); no longer U701.95 (GPIO52)
- net MCU_LCD_R7: now also U701.60 (GPIO30); no longer U701.98 (GPIO54)
Changed lines of the file:
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@@
 		)
 	)
-	(no_connect
-		(at 252.73 68.58)
+	(wire
+		(pts
+			(xy 252.73 68.58) (xy 247.65 68.58)
+		)
+		(stroke
+			(width 0)
+			(type default)
+		)
+	)
+	(hierarchical_label "MCU_LCD_R3"
+		(shape output)
+		(at 247.65 68.58 0)
+		(effects
+			(font
+				(size 0.8 0.8)
+			)
+			(justify right bottom)
+		)
 	)
 	(no_connect
 		(at 252.73 71.12)
 	)
-	(no_connect
-		(at 252.73 73.66)
+	(wire
+		(pts
+			(xy 252.73 73.66) (xy 247.65 73.66)
+		)
+		(stroke
+			(width 0)
+			(type default)
+		)
+	)
+	(hierarchical_label "MCU_LCD_R5"
+		(shape output)
+		(at 247.65 73.66 0)
+		(effects
+			(font
+				(size 0.8 0.8)
+			)
+			(justify right bottom)
+		)
 	)
 	(no_connect
 		(at 252.73 76.2)
 	)
-	(no_connect
-		(at 252.73 78.74)
+	(wire
+		(pts
+			(xy 252.73 78.74) (xy 247.65 78.74)
+		)
+		(stroke
+			(width 0)
+			(type default)
+		)
+	)
+	(hierarchical_label "MCU_LCD_R7"
+		(shape output)
+		(at 247.65 78.74 0)
+		(effects
+			(font
+				(size 0.8 0.8)
+			)
+			(justify right bottom)
+		)
 	)
 	(no_connect
 		(at 252.73 81.28)
 	)
-	(no_connect
-		(at 252.73 83.82)
+	(wire
+		(pts
+			(xy 252.73 83.82) (xy 247.65 83.82)
+		)
+		(stroke
+			(width 0)
+			(type default)
+		)
+	)
+	(hierarchical_label "MCU_LCD_G6"
+		(shape output)
+		(at 247.65 83.82 0)
+		(effects
+			(font
+				(size 0.8 0.8)
+			)
+			(justify right bottom)
+		)
 	)
 	(no_connect
@@
 		)
 	)
-	(wire
-		(pts
-			(xy 353.06 83.82) (xy 347.98 83.82)
-		)
-		(stroke
-			(width 0)
-			(type default)
-		)
-	)
-	(hierarchical_label "MCU_LCD_G6"
-		(shape output)
-		(at 347.98 83.82 0)
-		(effects
-			(font
-				(size 0.8 0.8)
-			)
-			(justify right bottom)
-		)
+	(no_connect
+		(at 353.06 83.82)
 	)
 	(wire
@@
 		)
 	)
-	(wire
-		(pts
-			(xy 453.39 59.69) (xy 448.31 59.69)
-		)
-		(stroke
-			(width 0)
-			(type default)
-		)
-	)
-	(hierarchical_label "MCU_LCD_R3"
-		(shape output)
-		(at 448.31 59.69 0)
-		(effects
-			(font
-				(size 0.8 0.8)
-			)
-			(justify right bottom)
-		)
+	(no_connect
+		(at 453.39 59.69)
 	)
 	(wire
@@
 		)
 	)
-	(wire
-		(pts
-			(xy 453.39 64.77) (xy 448.31 64.77)
-		)
-		(stroke
-			(width 0)
-			(type default)
-		)
-	)
-	(hierarchical_label "MCU_LCD_R5"
-		(shape output)
-		(at 448.31 64.77 0)
-		(effects
-			(font
-				(size 0.8 0.8)
-			)
-			(justify right bottom)
-		)
+	(no_connect
+		(at 453.39 64.77)
 	)
 	(wire
@@
 		)
 	)
-	(wire
-		(pts
-			(xy 453.39 69.85) (xy 448.31 69.85)
-		)
-		(stroke
-			(width 0)
-			(type default)
-		)
-	)
-	(hierarchical_label "MCU_LCD_R7"
-		(shape output)
-		(at 448.31 69.85 0)
-		(effects
-			(font
-				(size 0.8 0.8)
-			)
-			(justify right bottom)
-		)
-	)
-	(no_connect
+	(no_connect
+		(at 453.39 69.85)
+	)
+	(no_connect

Commit message: Complete all sixteen RGB resistor-to-FPC routes
Coordinate R4/R6 source GPIOs and underside poses with guarded source replacement. Add independently checked output topology, native clearance and preservation evidence, and current schematic/PCB review artifacts.
Connections:
- net MCU_LCD_R4: now also U701.56 (GPIO27); no longer U701.94 (GPIO51)
- net MCU_LCD_R6: now also U701.64 (GPIO33); no longer U701.97 (GPIO53)
Changed lines of the file:
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@@
 		)
 	)
-	(no_connect
-		(at 252.73 71.12)
+	(wire
+		(pts
+			(xy 252.73 71.12) (xy 247.65 71.12)
+		)
+		(stroke
+			(width 0)
+			(type default)
+		)
+	)
+	(hierarchical_label "MCU_LCD_R4"
+		(shape output)
+		(at 247.65 71.12 0)
+		(effects
+			(font
+				(size 0.8 0.8)
+			)
+			(justify right bottom)
+		)
 	)
 	(wire
@@
 		)
 	)
-	(no_connect
-		(at 353.06 45.72)
+	(wire
+		(pts
+			(xy 353.06 45.72) (xy 347.98 45.72)
+		)
+		(stroke
+			(width 0)
+			(type default)
+		)
+	)
+	(hierarchical_label "MCU_LCD_R6"
+		(shape output)
+		(at 347.98 45.72 0)
+		(effects
+			(font
+				(size 0.8 0.8)
+			)
+			(justify right bottom)
+		)
 	)
 	(wire
@@
 		(at 453.39 59.69)
 	)
-	(wire
-		(pts
-			(xy 453.39 62.23) (xy 448.31 62.23)
-		)
-		(stroke
-			(width 0)
-			(type default)
-		)
-	)
-	(hierarchical_label "MCU_LCD_R4"
-		(shape output)
-		(at 448.31 62.23 0)
-		(effects
-			(font
-				(size 0.8 0.8)
-			)
-			(justify right bottom)
-		)
+	(no_connect
+		(at 453.39 62.23)
 	)
 	(no_connect
 		(at 453.39 64.77)
 	)
-	(wire
-		(pts
-			(xy 453.39 67.31) (xy 448.31 67.31)
-		)
-		(stroke
-			(width 0)
-			(type default)
-		)
-	)
-	(hierarchical_label "MCU_LCD_R6"
-		(shape output)
-		(at 448.31 67.31 0)
-		(effects
-			(font
-				(size 0.8 0.8)
-			)
-			(justify right bottom)
-		)
-	)
-	(no_connect
+	(no_connect
+		(at 453.39 67.31)
+	)
+	(no_connect
