File: rev-b/generated/trials/display-timing.kicad_pcb (KiCad board)
At the start: 4 copper layers, 136 x 106 mm, 351 parts, among them J1001 LCD RGB / contact fit pending, J1002 CAP TOUCH / contact fit pendi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, J1101 FOOT WIRE: 1SIGNAL 2GND, J1102 FOOT WIRE: 1SIGNAL 2GND, J201 NMJ4HCD2 INPUT, J202 NMJ4HCD2 OUTPUT, J401 PJ-102AH, J501 GOWIN JTAG / target VREF only, J701 UART / POWERED TARGET ONLY, Q401 AO4407A, SW501 RECONFIG / MPN pending, SW701 RESET / SMD button MPN pending, SW702 BOOT / SMD button MPN pending, U101 TPS54302DDCR, U102 TPS54302DDCR, U1101 SN74LVC1G17DCKR, U1102 SN74LVC1G17DCKR, U201 PCM1808PWR, U202 PCM5102APWR, U203 OPA1656IDR, U204 TLV76750DRVR, U205 TLV75533PDBVR, U206 TPS3808G01DBVR, U207 TPS3808G01DBVR, U301 TLV62569DBVR, U302 TPS3897ADRYR, U303 TPS22965DSGR, U501 GW2AR-LV18QN88C8/I7, U502 GD25Q32ESIGR, U503 SN74LVC1G125DCKR, U504 SN74LVC1G17DCKR, U601 TLV62569DBVR, U701 ESP32-P4NRW16X, U702 GD25Q32ESIGR, U801 SN74AXC4T774PWR, U802 TPS3808G01DBVR, U803 SN74LVC1G00DCKR, U901 TPS61169DCKR, U902 SN74LVC1G125DCKR, U903 TLV76701DRVR, U904 TLV76701DRVR, Y501 24.576MHz / 3.3V CMOS XO / MP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, Y701 40MHz / +/-10ppm / MPN and CL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

Commit message: Preserve native-clear PCLK source and guarded trial courtyards
Parts:
- R1009, R1017, R1018: footprint Resistor_SMD:R_0402_1005Metric -> KestrelTiming:R_0402_1005Metric_Courtyard0p10
- moved R1017 3.75 mm to (122.7, 81.3)
Changed lines of the file:
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@@
 		)
 	)
-	(footprint "Resistor_SMD:R_0402_1005Metric"
+	(footprint "KestrelTiming:R_0402_1005Metric_Courtyard0p10"
 		(layer "B.Cu")
-		(at 118.9 81.2 90)
+		(at 122.65 81.3 90)
 		(descr "Resistor SMD 0402 (1005 Metric), square (rectangular) end terminal, IPC-7351 nominal, (Body size source: IPC-SM-782 page 72, https://www.pcb-3d.com/wordpress/wp-content/uploads/ipc-sm-782a_amendment_1_and_2.pdf)")
 		(tags "resistor")
@@
 				(font
 					(size 1.27 1.27)
-					(thickness 0.15)
 				)
 				(justify mirror)
@@
 				(font
 					(size 1.27 1.27)
-					(thickness 0.15)
 				)
 				(justify mirror)
@@
 				(font
 					(size 1.27 1.27)
-					(thickness 0.15)
 				)
 				(justify mirror)
@@
 				(font
 					(size 1.27 1.27)
-					(thickness 0.15)
 				)
 				(justify mirror)
@@
 		)
 		(property "AssemblySide" "B.Cu / source damping passives; assembly qualification pending"
-			(at 0 0 0)
+			(at 0 0 270)
 			(layer "B.SilkS")
 			(hide yes)
@@
 				(font
 					(size 1.27 1.27)
-					(thickness 0.15)
 				)
 				(justify mirror)
@@
 		)
 		(fp_rect
-			(start -0.93 0.47)
-			(end 0.93 -0.47)
+			(start -0.88 0.42)
+			(end 0.88 -0.42)
 			(stroke
 				(width 0.05)
@@
 		)
 	)
-	(footprint "Resistor_SMD:R_0402_1005Metric"
+	(footprint "KestrelTiming:R_0402_1005Metric_Courtyard0p10"
 		(layer "B.Cu")
-		(at 121.725 81.34 90)
+		(at 121.7 81.34 90)
 		(descr "Resistor SMD 0402 (1005 Metric), square (rectangular) end terminal, IPC-7351 nominal, (Body size source: IPC-SM-782 page 72, https://www.pcb-3d.com/wordpress/wp-content/uploads/ipc-sm-782a_amendment_1_and_2.pdf)")
 		(tags "resistor")
@@
 				(font
 					(size 1.27 1.27)
-					(thickness 0.15)
 				)
 				(justify mirror)
@@
 				(font
 					(size 1.27 1.27)
-					(thickness 0.15)
 				)
 				(justify mirror)
@@
 				(font
 					(size 1.27 1.27)
-					(thickness 0.15)
 				)
 				(justify mirror)
@@
 				(font
 					(size 1.27 1.27)
-					(thickness 0.15)
 				)
 				(justify mirror)
@@
 		)
 		(property "AssemblySide" "B.Cu / source damping passives; assembly qualification pending"
-			(at 0 0 0)
+			(at 0 0 270)
 			(layer "B.SilkS")
 			(hide yes)
@@
 				(font
 					(size 1.27 1.27)
-					(thickness 0.15)
 				)
 				(justify mirror)
@@
 		)
 		(fp_rect
-			(start -0.93 0.47)
-			(end 0.93 -0.47)
+			(start -0.88 0.42)
+			(end 0.88 -0.42)
 			(stroke
 				(width 0.05)
@@
 		)
 	)
-	(footprint "Resistor_SMD:R_0402_1005Metric"
+	(footprint "KestrelTiming:R_0402_1005Metric_Courtyard0p10"
 		(layer "B.Cu")
 		(at 123.6 80.4 90)
@@
 				(font
 					(size 1.27 1.27)
-					(thickness 0.15)
 				)
 			)
 		)
 		(property "Manufacturer" "YAGEO"
-			(at 0 0 0)
+			(at 0 0 270)
 			(layer "B.SilkS")
 			(hide yes)
@@
 				(font
 					(size 1.27 1.27)
-					(thickness 0.15)
 				)
 			)
 		)
 		(property "MPN" "RC0402FR-0733RL"
-			(at 0 0 0)
+			(at 0 0 270)
 			(layer "B.SilkS")
 			(hide yes)
@@
 				(font
 					(size 1.27 1.27)
-					(thickness 0.15)
 				)
 			)
 		)
 		(property "LCSC" "C138002"
-			(at 0 0 0)
+			(at 0 0 270)
 			(layer "B.SilkS")
 			(hide yes)
@@
 				(font
 					(size 1.27 1.27)
-					(thickness 0.15)
 				)
 			)
 		)
 		(property "Rating" "33ohm / 1% / 0.063W at 70C / 50V limiting voltage / GPIO source damping starting value"
-			(at 0 0 0)
+			(at 0 0 270)
 			(layer "B.SilkS")
 			(hide yes)
@@
 				(font
 					(size 1.27 1.27)
-					(thickness 0.15)
 				)
 			)
@@
 		)
 		(fp_rect
-			(start -0.93 0.47)
-			(end 0.93 -0.47)
+			(start -0.88 0.42)
+			(end 0.88 -0.42)
 			(stroke
 				(width 0.05)
